File: rpi-aeroguard-template_v4/cm4-high-speed.kicad_sch (KiCad schematic)
At the start: 2 parts, among them J1 F305-1A7H1-21022-E100

Commit message: Add files via upload
Parts:
- removed Module1: ComputeModule4-CM4, CM4IO:Raspberry-Pi-4-Compute-Module, symbol CM4IO:ComputeModule4-CM4
- added J7: DF40C-100DS-0.4V_51_, DF40C-100DS-0.4V_51_:HIROSE_DF40C-100DS-0.4V_51_, symbol DF40C-100DS-0.4V_51_:DF40C-100DS-0.4V_51_
Connections:
- net CAM0_C_N: now also J7.27
- net CAM0_C_P: now also J7.29
- net CAM0_D0_N: now also J7.15
- net CAM0_D0_P: now also J7.17
- net CAM0_D1_N: now also J7.21
- net CAM0_D1_P: now also J7.23
- net GND: now also J7.13, J7.14, J7.19, J7.20, J7.25, J7.26, J7.31, J7.32, J7.37, J7.38, J7.44, J7.50, J7.55, J7.56, J7.61, J7.62, J7.67, J7.68, J7.7, J7.73, J7.74, J7.79, J7.8, J7.80, J7.85, J7.86, J7.91, J7.92, J7.97, J7.98
