File: rpi-aeroguard-template_v4/rpi-cm4-carrier-template.kicad_pcb (KiCad board)
At the start: 2 copper layers, 40 x 55 mm, 32 parts, among them J1 F305-1A7H1-21022-E100, J2 Conn_01x02_Pin, J3 Conn_01x04_Pin, J4 Conn_01x02_Pin, J6 Conn_01x05_Pin, U1 TPS63070RNMR, U2 74LVC1G07SE-7

Commit message: Add files via upload
Parts:
- removed D4: LED, LED_THT:LED_D1.8mm_W3.3mm_H2.4mm
- removed Module1: ComputeModule4-CM4, CM4IO:Raspberry-Pi-4-Compute-Module
- removed R8: DNF, Resistor_THT:R_Axial_DIN0204_L3.6mm_D1.6mm_P5.08mm_Horizontal
- added J5: DF40C-100DS-0.4V_51_, DF40C-100DS-0.4V_51_:HIROSE_DF40C-100DS-0.4V_51_, F.Cu at (163.5, 102.8)
- added J7: DF40C-100DS-0.4V_51_, DF40C-100DS-0.4V_51_:HIROSE_DF40C-100DS-0.4V_51_, F.Cu at (129.5, 102.8)
- moved R2 140.3 mm to (191.1, 107.5), turned to 180 degrees
- moved LS1 135.2 mm to (175.5, 116.5), turned to 180 degrees
- moved R10 132.5 mm to (176.5, 137.5), turned to 180 degrees
- moved J3 132.4 mm to (187.8, 121.3)
- moved R9 131.5 mm to (178.0, 129.0), turned to 180 degrees
- moved U1 124.8 mm to (181.2, 86.6)
- moved R4 121.3 mm to (179.9, 72.0)
- moved R1 119.3 mm to (169.0, 103.5)
- moved R5 118.6 mm to (174.0, 98.5), turned to 180 degrees
- moved R3 113.6 mm to (169.0, 91.5)
- moved J4 103.4 mm to (170.0, 85.0), turned to 180 degrees
- moved L1 103.2 mm to (175.0, 86.9), turned to -90 degrees
- moved C6 102.7 mm to (181.4, 104.0)
- moved C2 95.8 mm to (188.0, 99.5)
- moved C8 92.2 mm to (181.4, 93.0)
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Routing:
- net /CM4 GPIO/GPIO19: track 0.00 -> 124.1 mm
- net GND: track 0.00 -> 104.7 mm
- net /CM4 GPIO/GPIO18: track 0.00 -> 72.8 mm
- net +5V: track 0.00 -> 61.9 mm
- net /CM4 GPIO/nPWR_LED: track 0.00 -> 60.3 mm
- net VIN: track 0.00 -> 55.2 mm
- net /CM4 GPIO/GPIO 5: track 0.00 -> 37.9 mm
- net /CM4 GPIO/GPIO 13: track 0.00 -> 28.7 mm
- net /CM4 GPIO/GPIO17: track 0.00 -> 27.4 mm
- net Net-(J3-Pin_4): track 0.00 -> 25.9 mm
- net /CM4 GPIO/GPIO 12: track 0.00 -> 21.4 mm
- net FB: track 0.00 -> 18.8 mm
- net Net-(J3-Pin_1): track 0.00 -> 12.1 mm
- net Net-(D2-K): track 0.00 -> 11.9 mm
- net +3.3V: track 0.00 -> 11.9 mm
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Other:
- board outline removed
- board text removed: "Receptacle component options: 1.5mm height: 2x Hirose DF40C-100DS-0.4v OR 3.0mm height: 2x Hirose DF40HC(3.0)-100DS-0.4v"

Commit message: Add files via upload
Parts:
- moved LS1 45.3 mm to (133.8, 134.3)
- moved R4 44.1 mm to (176.1, 115.9)
- moved J3 44.0 mm to (145.7, 133.9), turned to 90 degrees
- moved C3 22.1 mm to (178.1, 106.2)
- moved R2 22.0 mm to (169.5, 111.7), turned to 90 degrees
- moved R9 21.2 mm to (157.9, 135.7), turned to 90 degrees
- moved C1 20.2 mm to (178.1, 111.5)
- moved C7 16.3 mm to (178.1, 103.4)
- moved C2 13.7 mm to (178.1, 109.0)
- moved L1 13.5 mm to (184.6, 96.4)
- moved R10 13.4 mm to (163.2, 135.8), turned to 90 degrees
- moved C5 13.1 mm to (179.8, 85.5), turned to 0 degrees
- moved U2 9.40 mm to (124.7, 87.4)
- moved R6 6.73 mm to (117.0, 87.5)
- moved C4 6.67 mm to (184.4, 85.6)
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Connections:
- J3 pad 2: /CM4 GPIO/3.3V -> +3.3V
Routing:
- net GND: track 104.7 -> 319.3 mm, vias 0 -> 59
- net +3.3V: track 11.9 -> 101.8 mm, vias 0 -> 5
- net /CM4 GPIO/PI_nLED_Activity: track 0.00 -> 67.5 mm, vias 0 -> 1
- net /CM4 GPIO/GPIO21: track 0.00 -> 65.7 mm, vias 0 -> 7
- net /CM4 High Speed/SCL1: track 0.00 -> 63.8 mm, vias 0 -> 2
- net /CM4 High Speed/SDA1: track 0.00 -> 63.7 mm
- net /CM4 GPIO/GPIO18: track 72.8 -> 126.5 mm, vias 0 -> 2
- net Net-(J3-Pin_1): track 12.1 -> 49.7 mm
- net EN: track 0.00 -> 35.4 mm, vias 0 -> 2
- net /CM4 High Speed/CAM0_C_P: track 0.00 -> 27.8 mm
- net /CM4 High Speed/CAM0_C_N: track 0.00 -> 26.3 mm
- net /CM4 GPIO/GPIO17: track 27.4 -> 53.6 mm, vias 0 -> 2
- net /CM4 High Speed/CAM0_D1_P: track 0.00 -> 24.1 mm
- net /CM4 High Speed/CAM0_D1_N: track 0.00 -> 22.8 mm
- net /CM4 High Speed/CAM0_D0_P: track 0.00 -> 20.9 mm
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- added copper zone on B.Cu, net GND
- added copper zone on F.Cu, net GND
Other:
- board outline added: 73.9 x 57.7 mm
- board text removed: "Wireless Keepout"
- board text removed: "v01"
